File: WCH/KiCAD/SignalGenerator/SignalGenerator/signalgenerator-rounded.kicad_pcb (KiCad board)
At the start: 2 copper layers, 78 x 57 mm, 29 parts, among them J1 Conn_01x10, J2 Conn_01x10, J3 Conn_02x05_Odd_Even, J4 Conn_01x02, J5 Conn_01x07_Pin, J6 Conn_Coaxial, J7 Conn_01x12, J8 Conn_01x12, J9 Conn_01x12, U1 CH32V003F4P6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

Commit message: PCB
Parts:
- removed the REF** at (36.2, 67.3)
- added 1: PC1, TestPoint:TestPoint_Pad_D2.0mm, B.Cu at (61.6, 69.8)
- added 3: PC1, TestPoint:TestPoint_Pad_D2.0mm, B.Cu at (61.6, 74.9)
- added 5: PC1, TestPoint:TestPoint_Pad_D2.0mm, B.Cu at (45.7, 74.9)
- added 6: PC1, TestPoint:TestPoint_Pad_D2.0mm, B.Cu at (48.3, 73.0)
- added 7: PC1, TestPoint:TestPoint_Pad_D2.0mm, B.Cu at (45.7, 71.1)
- added 8: PC1, TestPoint:TestPoint_Pad_D2.0mm, B.Cu at (48.3, 69.2)
- added D1: SK6805, LED_SMD:LED_SK6812_EC15_1.5x1.5mm, B.Cu at (65.0, 72.6)
- added U4: CH32V003J4M6, Package_SO:SOIC-8_3.9x4.9mm_P1.27mm, B.Cu at (54.6, 72.4)
- moved R5 49.7 mm to (80.8, 67.7)
- moved SW5 48.4 mm to (84.7, 75.3)
- moved R1 30.9 mm to (33.0, 67.3), turned to 90 degrees
- moved SW2 21.8 mm to (70.5, 75.3)
- moved SW1 20.5 mm to (57.7, 66.4), turned to 180 degrees
- moved R4 18.8 mm to (36.8, 67.3), turned to 90 degrees
- moved R3 15.4 mm to (40.6, 67.3), turned to 90 degrees
- moved R2 11.1 mm to (66.5, 67.7)
- moved SW3 10.0 mm to (45.1, 75.3)
- moved SW4 4.53 mm to (57.8, 75.3)
- renumbered UP to SW1, DOWN to SW2, LEFT to SW3, RIGHT to SW4, ENTER to SW5
Routing:
- net /SWDIO: track 41.6 -> 93.2 mm
- net /UP: track 60.4 -> 92.9 mm
- net +3.3V: track 277.0 -> 303.5 mm
- net J9_12: track 0.00 -> 23.3 mm
- net /DOWN: track 68.8 -> 54.5 mm
- net /RIGHT: track 56.5 -> 68.2 mm
- net Net-(D1-DIN): track 0.00 -> 8.33 mm
- net /LEFT: track 39.7 -> 47.9 mm
- net /ENTER: track 65.6 -> 58.5 mm
- net Net-(U4-PC1): track 0.00 -> 6.57 mm
- net Net-(U4-PC4): track 0.00 -> 6.57 mm
- net Net-(U4-PA2): track 0.00 -> 5.15 mm
- net Net-(U4-PC2): track 0.00 -> 3.88 mm
- net GND: track 347.8 -> 344.7 mm
- net +5V: track 43.7 -> 44.4 mm
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